File: elec/QRD.sch (EAGLE design)
At the start: 7 parts, among them IC1 LM311D

Commit message: modified QRD added potentialmeter value
Parts:
- R4: value (none) -> 100k
Changed lines of the file:
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@@
 <part name="R3" library="resistor" deviceset="R-US_" device="0204/2V" value="47k"/>
 <part name="IC1" library="linear" deviceset="LM311" device="D"/>
-<part name="R4" library="pot" deviceset="TRIM_US-" device="3223G"/>
+<part name="R4" library="pot" deviceset="TRIM_US-" device="3223G" value="100k"/>
 </parts>
 <sheets>
